File: interconnect.kicad_sch (KiCad schematic)
At the start: 6 parts, among them J1 Conn_02x04_Odd_Even, J2 Conn_02x04_Odd_Even, X1 NUCLEO144-ZIO

Commit message: Add files via upload
Parts:
- FB1, FB2, FB3: footprint (none) -> Inductor_SMD:L_0805_2012Metric
Other:
- moved on the sheet: FB1, FB2, FB3, J1, J2
