File: NR1B-analog.kicad_pcb (KiCad board)
At the start: 4 copper layers, 71.1 x 134.5 mm, 64 parts, among them J1 Conn_02x04_Odd_Even, J2 Conn_02x04_Odd_Even, J3 Conn_01x03_Male, J8 Conn_01x04_Male, SW1 1-1571636-0, U1 DAC11001BPFBR, U10 LT3042MPMSE-PBF, U11 LDK320ADU120R, U12 20K, U13 OPA2189IDR, U14 DAC11001BPFBR, U2 ADR444ARZ, U3 OPA189IDGKT, U4 OPA2189IDR, U5 Pico, U7 LT3093EMSE-PBF, U8 20K, U9 10K, X1 NUCLEO144-ZIO

Commit message: Add files via upload
Parts:
- added CS_DAC0: TestPoint, TestPoint:TestPoint_Bridge_Pitch2.0mm_Drill0.7mm, F.Cu at (80.9, 80.7)
- added CS_DAC1: TestPoint, TestPoint:TestPoint_Bridge_Pitch2.0mm_Drill0.7mm, F.Cu at (80.9, 83.3)
- added CS_SYS1: TestPoint, TestPoint:TestPoint_Bridge_Pitch2.0mm_Drill0.7mm, F.Cu at (101.8, 109.0)
- added GND: TestPoint, TestPoint:TestPoint_Bridge_Pitch2.0mm_Drill0.7mm, F.Cu at (80.9, 85.8)
- added MISO_DAC1: TestPoint, TestPoint:TestPoint_Bridge_Pitch2.0mm_Drill0.7mm, F.Cu at (80.9, 75.6)
- added MISO_SYS1: TestPoint, TestPoint:TestPoint_Bridge_Pitch2.0mm_Drill0.7mm, F.Cu at (101.8, 103.9)
- added MOSI_DAC1: TestPoint, TestPoint:TestPoint_Bridge_Pitch2.0mm_Drill0.7mm, F.Cu at (80.9, 78.2)
- added MOSI_SYS1: TestPoint, TestPoint:TestPoint_Bridge_Pitch2.0mm_Drill0.7mm, F.Cu at (101.8, 106.4)
- added SCK_DAC1: TestPoint, TestPoint:TestPoint_Bridge_Pitch2.0mm_Drill0.7mm, F.Cu at (80.9, 73.1)
- added SCK_SYS1: TestPoint, TestPoint:TestPoint_Bridge_Pitch2.0mm_Drill0.7mm, F.Cu at (101.8, 101.3)
- added TP1: TestPoint, TestPoint:TestPoint_Bridge_Pitch2.0mm_Drill0.7mm, F.Cu at (102.4, 131.6)
- added TP2: TestPoint, TestPoint:TestPoint_Bridge_Pitch2.0mm_Drill0.7mm, F.Cu at (102.4, 129.0)
- added TP3: TestPoint, TestPoint:TestPoint_Bridge_Pitch2.0mm_Drill0.7mm, F.Cu at (66.2, 109.1)
- added TP4: TestPoint, TestPoint:TestPoint_Bridge_Pitch2.0mm_Drill0.7mm, F.Cu at (66.2, 111.6)
- added TP5: TestPoint, TestPoint:TestPoint_Bridge_Pitch2.0mm_Drill0.7mm, F.Cu at (66.2, 114.1)
- added TP6: TestPoint, TestPoint:TestPoint_Bridge_Pitch2.0mm_Drill0.7mm, F.Cu at (66.2, 116.7)
- added TP7: TestPoint, TestPoint:TestPoint_Bridge_Pitch2.0mm_Drill0.7mm, F.Cu at (66.2, 119.2)
- added TP8: TestPoint, TestPoint:TestPoint_Bridge_Pitch2.0mm_Drill0.7mm, F.Cu at (66.2, 121.8)
- moved C20 1.05 mm to (94.9, 72.5)
Routing:
- net /Interconnect/MOSI: track 72.4 -> 106.7 mm, vias 0 -> 3
- net /Interconnect/NSS: track 70.6 -> 101.4 mm, vias 0 -> 1
- net Net-(TP8-Pad1): track 0.00 -> 19.4 mm
- net Net-(TP2-Pad1): track 0.00 -> 19.0 mm
- net Net-(TP1-Pad1): track 0.00 -> 18.4 mm
- net /MCU/CS_DAC0: track 57.5 -> 75.6 mm, vias 0 -> 1
- net /MCU/MOSI_DAC: track 77.3 -> 95.2 mm, vias 3 -> 5
- net Net-(TP7-Pad1): track 0.00 -> 16.9 mm
- net Net-(TP6-Pad1): track 0.00 -> 16.9 mm
- net Net-(TP5-Pad1): track 0.00 -> 14.4 mm
- net /MCU/SCK_DAC: track 81.4 -> 95.7 mm, vias 2 -> 4
- net /MCU/MISO_DAC: track 88.2 -> 102.2 mm
- net Net-(TP4-Pad1): track 0.00 -> 13.0 mm
- net Net-(TP3-Pad1): track 0.00 -> 13.0 mm
- net /MCU/CS_DAC1: track 52.7 -> 62.8 mm
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Other:
- board text added: "3V3"
- board text added: "CLK"
- board text added: "GND"
- board text added: "RX"
- board text added: "SWD"
- board text added: "TX"
