File: NR1B-analog.kicad_sch (KiCad schematic)
At the start: 54 parts, among them U1 DAC11001BPFBR, U10 LT3042MPMSE-PBF, U11 LDK320ADU120R, U12 20K, U13 OPA2189IDR, U14 DAC11001BPFBR, U2 ADR444ARZ, U3 OPA189IDGKT, U4 OPA2189IDR, U7 LT3093EMSE-PBF, U8 20K, U9 10K

Commit message: Add files via upload
Parts:
- removed C14: 0.1uF, Capacitor_SMD:C_0603_1608Metric, symbol Device:C
- removed C42, C44: 2.2uF, Capacitor_SMD:C_0805_2012Metric, symbol Device:C_Polarized
- added C22, C23: 2.2uF, Capacitor_SMD:C_0603_1608Metric, symbol Device:C
- added J8: Conn_01x04_Male, Connector_PinHeader_2.54mm:PinHeader_1x04_P2.54mm_Horizontal, symbol Connector:Conn_01x04_Male
- C12, C13, C2, C5, C7: footprint (none) -> Capacitor_SMD:CP_Elec_5x5.3
Connections:
- net +14Vreg: now also C10.2, U11.2 (IN)
- net +15Vreg: no longer C10.2, U11.2 (IN)
- net +3V3: now also J8.4 (Pin_4)
- net +5V: now also C22.1, C23.1
- net GND: now also C22.2, C23.2, J8.1 (Pin_1)
- new net MCU/UART_RX: J8.3 (Pin_3)
- new net MCU/UART_TX: J8.2 (Pin_2)
Other:
- sheet MCU ports: added UART_RX, UART_TX; removed none

Commit message: Add files via upload
Parts:
- added CS_DAC0, CS_DAC1, CS_SYS1, GND1, MISO_DAC1, MISO_SYS1, MOSI_DAC1, MOSI_SYS1, SCK_DAC1, SCK_SYS1: TestPoint, TestPoint:TestPoint_Bridge_Pitch2.0mm_Drill0.7mm, symbol Connector:TestPoint
Connections:
- net GND: now also GND1.1
- net Interconnect/MISO: now also MISO_SYS1.1
- net Interconnect/MOSI: now also MOSI_SYS1.1
- net Interconnect/NSS: now also CS_SYS1.1
- net Interconnect/SCK: now also SCK_SYS1.1
- net MCU/CS_DAC0: now also CS_DAC0.1
- net MCU/CS_DAC1: now also CS_DAC1.1
- net MCU/MISO_DAC: now also MISO_DAC1.1
- net MCU/MOSI_DAC: now also MOSI_DAC1.1
- net MCU/SCK_DAC: now also SCK_DAC1.1
