File: NR1B-Power/NR1B-Power.kicad_pcb (KiCad board)
At the start: 4 copper layers, 70.5 x 134 mm, 43 parts, among them J1 Conn_02x04_Odd_Even, J2 Conn_02x04_Odd_Even, J3 3.81mm Pluggable Terminal, U1 TSR_1-2450, U2 DKMW06, U3 VO615A, U4 VO615A, X1 NUCLEO144-ZIO

Commit message: Added Manufacturers and part numbers
Parts:
- J1, J2: value Conn_02x04_Odd_Even -> 0.1" Female long-tail
Changed lines of the file:
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@@
     (descr "Through hole straight pin header, 2x04, 2.54mm pitch, double rows")
     (tags "Through hole pin header THT 2x04 2.54mm double row")
+    (property "MFG 1" "Mill-Max")
+    (property "MPN 1" "411-XX-2XX-41-001000")
     (property "Sheetfile" "NR1B-Power.kicad_sch")
     (property "Sheetname" "")
@@
       (effects (font (size 1 1) (thickness 0.15)))
     )
-    (fp_text value "Conn_02x04_Odd_Even" (at 1.27 9.95) (layer "F.Fab")
+    (fp_text value "0.1\" Female long-tail" (at 1.27 9.95) (layer "F.Fab")
       (effects (font (size 1 1) (thickness 0.15)))
     )
@@
     (descr "4-lead though-hole mounted DIP package, row spacing 7.62 mm (300 mils), LongPads")
     (tags "THT DIP DIL PDIP 2.54mm 7.62mm 300mil LongPads")
+    (property "MFG 1" "Vishay")
+    (property "MPN 1" "VO615A")
     (property "Sheetfile" "NR1B-Power.kicad_sch")
     (property "Sheetname" "")
@@
     (descr "Fuse SMD 1812 (4532 Metric), square (rectangular) end terminal, IPC_7351 nominal, (Body size source: https://www.nikhef.nl/pub/departments/mt/projects/detectorR_D/dtddice/ERJ2G.pdf), generated with kicad-footprint-generator")
     (tags "fuse")
+    (property "MFG 1" "Bel Fuse")
+    (property "MPN 1" "0ZCG0030FF2C")
     (property "Sheetfile" "NR1B-Power.kicad_sch")
     (property "Sheetname" "")
@@
     (descr "DCDC-Converter, TRACO, TSR 1-xxxx")
     (tags "DCDC-Converter TRACO TSR-1")
+    (property "MFG 1" "TRACO")
+    (property "MPN 1" "TSR 1-2450")
     (property "Sheetfile" "NR1B-Power.kicad_sch")
     (property "Sheetname" "")
@@
     (descr "DCDC-Converter, Meanwell, DKMW06, dual output")
     (tags "DCDC-Converter Meanwell DKMW06 dual output")
+    (property "MFG 1" "Mean Well")
+    (property "MPN 1" "DKMW06F-15")
     (property "Sheetfile" "NR1B-Power.kicad_sch")
     (property "Sheetname" "")
@@
     (descr "Generic Phoenix Contact connector footprint for: MC_1,5/2-G-3.5; number of pins: 02; pin pitch: 3.50mm; Angled || order number: 1844210 8A 160V")
     (tags "phoenix_contact connector MC_01x02_G_3.5mm")
+    (property "MFG 1" "CUI")
+    (property "MPN 1" "TBP03R1-350-02BE")
     (property "Sheetfile" "NR1B-Power.kicad_sch")
     (property "Sheetname" "")
@@
     (descr "LED SMD 0805 (2012 Metric), square (rectangular) end terminal, IPC_7351 nominal, (Body size source: https://docs.google.com/spreadsheets/d/1BsfQQcO9C6DZCsRaXUlFlo91Tg2WpOkGARC1WS5S8t0/edit?usp=sharing), generated with kicad-footprint-generator")
     (tags "LED")
-    (property "MPN" "APT2012LZGCK")
+    (property "MPN" "APT2012LSECK/J3-PRV")
     (property "Manufacturer" "Kingbright")
     (property "Sheetfile" "NR1B-Power.kicad_sch")
@@
     (descr "LED SMD 0805 (2012 Metric), square (rectangular) end terminal, IPC_7351 nominal, (Body size source: https://docs.google.com/spreadsheets/d/1BsfQQcO9C6DZCsRaXUlFlo91Tg2WpOkGARC1WS5S8t0/edit?usp=sharing), generated with kicad-footprint-generator")
     (tags "LED")
-    (property "MPN" "APT2012LZGCK")
+    (property "MPN" "APT2012LSECK/J3-PRV")
     (property "Manufacturer" "Kingbright")
     (property "Sheetfile" "NR1B-Power.kicad_sch")
@@
     (descr "Through hole straight pin header, 2x04, 2.54mm pitch, double rows")
     (tags "Through hole pin header THT 2x04 2.54mm double row")
+    (property "MFG 1" "Mill-Max")
+    (property "MPN 1" "411-XX-2XX-41-001000")
     (property "Sheetfile" "NR1B-Power.kicad_sch")
     (property "Sheetname" "")
@@
       (effects (font (size 1 1) (thickness 0.15)))
     )
-    (fp_text value "Conn_02x04_Odd_Even" (at 1.27 9.95) (layer "F.Fab")
+    (fp_text value "0.1\" Female long-tail" (at 1.27 9.95) (layer "F.Fab")
       (effects (font (size 1 1) (thickness 0.15)))
     )
@@
     (descr "4-lead though-hole mounted DIP package, row spacing 7.62 mm (300 mils), LongPads")
     (tags "THT DIP DIL PDIP 2.54mm 7.62mm 300mil LongPads")
-    (property "Sheetfile" "NR1B-Power.kicad_sch")
-    (property "Sheetname" "")
+    (property "MFG 1" "Vishay")
+    (property "MPN 1" "VO615A")
+    (property "Sheetfile" "NR1B-Power.kicad_sch")
+    (property "Sheetname" "")

Commit message: Changed C1
Parts:
- C1: value 47uF -> 47uF 50V; footprint Capacitor_SMD:CP_Elec_5x5.3 -> Capacitor_SMD:CP_Elec_6.3x7.7
- C2: value 47uF -> 47uF 16V
- moved C1 0.75 mm to (209.0, 100.8)

Commit message: Fixed footprints
Parts:
- D1: footprint Diode_SMD:D_SOD-323 -> Diode_SMD:D_SMA
- moved D1 1.36 mm to (218.6, 100.4), turned to 0 degrees
- moved D2 1.35 mm to (213.9, 101.8)
Routing:
- net Net-(D1-Pad2): track 8.83 -> 9.85 mm
Changed lines of the file:
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@@
     )
   )
-  (footprint "Diode_SMD:D_SOD-323" (layer "F.Cu")
-    (at 218.75 101.75 90)
-    (descr "SOD-323")
-    (tags "SOD-323")
+  (footprint "Diode_SMD:D_SMA" (layer "F.Cu")
+    (at 218.6 100.4)
+    (descr "Diode SMA (DO-214AC)")
+    (tags "Diode SMA (DO-214AC)")
     (property "Sheetfile" "NR1B-Power.kicad_sch")
     (property "Sheetname" "")
     (attr smd)
-    (fp_text reference "D1" (at 0.25 1.75 90) (layer "F.SilkS")
-      (effects (font (size 1 1) (thickness 0.15)))
-    )
-    (fp_text value "S1G" (at 0 -1.75 90) (layer "F.Fab")
-      (effects (font (size 1 1) (thickness 0.15)))
-    )
-    (fp_text user "${REFERENCE}" (at 0.25 1.75 90) (layer "F.Fab")
-      (effects (font (size 1 1) (thickness 0.15)))
-    )
-    (fp_line (start -1.5 -0.85) (end -1.5 0.85) (layer "F.SilkS") (width 0.12))
-    (fp_line (start -1.5 -0.85) (end 1.05 -0.85) (layer "F.SilkS") (width 0.12))
-    (fp_line (start -1.5 0.85) (end 1.05 0.85) (layer "F.SilkS") (width 0.12))
-    (fp_line (start -1.6 -0.95) (end -1.6 0.95) (layer "F.CrtYd") (width 0.05))
-    (fp_line (start 1.6 -0.95) (end 1.6 0.95) (layer "F.CrtYd") (width 0.05))
-    (fp_line (start -1.6 0.95) (end 1.6 0.95) (layer "F.CrtYd") (width 0.05))
-    (fp_line (start -1.6 -0.95) (end 1.6 -0.95) (layer "F.CrtYd") (width 0.05))
-    (fp_line (start 0.9 0.7) (end -0.9 0.7) (layer "F.Fab") (width 0.1))
-    (fp_line (start 0.9 -0.7) (end 0.9 0.7) (layer "F.Fab") (width 0.1))
-    (fp_line (start 0.2 0.35) (end -0.3 0) (layer "F.Fab") (width 0.1))
-    (fp_line (start 0.2 0) (end 0.45 0) (layer "F.Fab") (width 0.1))
-    (fp_line (start -0.3 0) (end 0.2 -0.35) (layer "F.Fab") (width 0.1))
-    (fp_line (start -0.9 -0.7) (end 0.9 -0.7) (layer "F.Fab") (width 0.1))
-    (fp_line (start -0.9 0.7) (end -0.9 -0.7) (layer "F.Fab") (width 0.1))
-    (fp_line (start 0.2 -0.35) (end 0.2 0.35) (layer "F.Fab") (width 0.1))
-    (fp_line (start -0.3 -0.35) (end -0.3 0.35) (layer "F.Fab") (width 0.1))
-    (fp_line (start -0.3 0) (end -0.5 0) (layer "F.Fab") (width 0.1))
-    (pad "1" smd rect (at -1.05 0 90) (size 0.6 0.45) (layers "F.Cu" "F.Paste" "F.Mask")
+    (fp_text reference "D1" (at 2.5 2.6) (layer "F.SilkS")
+      (effects (font (size 1 1) (thickness 0.15)))
+    )
+    (fp_text value "S1G" (at 0 2.6) (layer "F.Fab")
+      (effects (font (size 1 1) (thickness 0.15)))
+    )
+    (fp_text user "${REFERENCE}" (at 0 -2.5) (layer "F.Fab")
+      (effects (font (size 1 1) (thickness 0.15)))
+    )
+    (fp_line (start -3.4 1.65) (end 2 1.65) (layer "F.SilkS") (width 0.12))
+    (fp_line (start -3.4 -1.65) (end -3.4 1.65) (layer "F.SilkS") (width 0.12))
+    (fp_line (start -3.4 -1.65) (end 2 -1.65) (layer "F.SilkS") (width 0.12))
+    (fp_line (start -3.5 -1.75) (end 3.5 -1.75) (layer "F.CrtYd") (width 0.05))
+    (fp_line (start 3.5 1.75) (end -3.5 1.75) (layer "F.CrtYd") (width 0.05))
+    (fp_line (start 3.5 -1.75) (end 3.5 1.75) (layer "F.CrtYd") (width 0.05))
+    (fp_line (start -3.5 1.75) (end -3.5 -1.75) (layer "F.CrtYd") (width 0.05))
+    (fp_line (start 2.3 1.5) (end -2.3 1.5) (layer "F.Fab") (width 0.1))
+    (fp_line (start 0.50118 0.75032) (end 0.50118 -0.79908) (layer "F.Fab") (width 0.1))
+    (fp_line (start -2.3 1.5) (end -2.3 -1.5) (layer "F.Fab") (width 0.1))
+    (fp_line (start 0.50118 0.00102) (end 1.4994 0.00102) (layer "F.Fab") (width 0.1))
+    (fp_line (start -0.64944 0.00102) (end 0.50118 0.75032) (layer "F.Fab") (width 0.1))
+    (fp_line (start 2.3 -1.5) (end -2.3 -1.5) (layer "F.Fab") (width 0.1))
+    (fp_line (start -0.64944 0.00102) (end -1.55114 0.00102) (layer "F.Fab") (width 0.1))
+    (fp_line (start -0.64944 -0.79908) (end -0.64944 0.80112) (layer "F.Fab") (width 0.1))
+    (fp_line (start 2.3 -1.5) (end 2.3 1.5) (layer "F.Fab") (width 0.1))
+    (fp_line (start -0.64944 0.00102) (end 0.50118 -0.79908) (layer "F.Fab") (width 0.1))
+    (pad "1" smd rect (at -2 0) (size 2.5 1.8) (layers "F.Cu" "F.Paste" "F.Mask")
       (net 6 "+24V") (pinfunction "K") (pintype "passive"))
-    (pad "2" smd rect (at 1.05 0 90) (size 0.6 0.45) (layers "F.Cu" "F.Paste" "F.Mask")
+    (pad "2" smd rect (at 2 0) (size 2.5 1.8) (layers "F.Cu" "F.Paste" "F.Mask")
       (net 48 "Net-(D1-Pad2)") (pinfunction "A") (pintype "passive"))
-    (model "${KICAD6_3DMODEL_DIR}/Diode_SMD.3dshapes/D_SOD-323.wrl"
+    (model "${KICAD6_3DMODEL_DIR}/Diode_SMD.3dshapes/D_SMA.wrl"
       (offset (xyz 0 0 0))
       (scale (xyz 1 1 1))
@@
   )
   (footprint "Diode_SMD:D_SOD-323" (layer "F.Cu")
-    (at 215.25 101.75 90)
+    (at 213.9 101.75 90)
     (descr "SOD-323")
     (tags "SOD-323")
@@
     (property "Sheetname" "")
     (attr smd)
-    (fp_text reference "D2" (at 0 -1.85 90) (layer "F.SilkS")
+    (fp_text reference "D2" (at -1.35 2 180) (layer "F.SilkS")
       (effects (font (size 1 1) (thickness 0.15)))
     )
@@
   (via (at 183.75 210.25) (size 0.8) (drill 0.4) (layers "F.Cu" "B.Cu") (net 8))
   (via (at 192.75 92) (size 0.8) (drill 0.4) (layers "F.Cu" "B.Cu") (free) (net 8))
-  (via (at 215.75 99.5) (size 0.8) (drill 0.4) (layers "F.Cu" "B.Cu") (free) (net 8))
+  (via (at 214.4 99.5) (size 0.8) (drill 0.4) (layers "F.Cu" "B.Cu") (free) (net 8))
   (via (at 207 97.75) (size 0.8) (drill 0.4) (layers "F.Cu" "B.Cu") (free) (net 8))
   (via (at 196.5 89.25) (size 0.8) (drill 0.4) (layers "F.Cu" "B.Cu") (free) (net 8))
   (via (at 178.5 161.5) (size 0.8) (drill 0.4) (layers "F.Cu" "B.Cu") (free) (net 8))
   (via (at 182.5 161.5) (size 0.8) (drill 0.4) (layers "F.Cu" "B.Cu") (free) (net 8))
-  (via (at 214.75 99.5) (size 0.8) (drill 0.4) (layers "F.Cu" "B.Cu") (free) (net 8))
+  (via (at 213.4 99.5) (size 0.8) (drill 0.4) (layers "F.Cu" "B.Cu") (free) (net 8))
   (via (at 179.75 161.5) (size 0.8) (drill 0.4) (layers "F.Cu" "B.Cu") (free) (net 8))
   (via (at 211 95.25) (size 0.8) (drill 0.4) (layers "F.Cu" "B.Cu") (free) (net 8))
@@
   (segment (start 182.84 93.66) (end 183.25 93.25) (width 0.4) (layer "B.Cu") (net 21))
   (segment (start 219.25 178) (end 202 195.25) (width 0.4) (layer "B.Cu") (net 21))
-  (segment (start 215.75 95) (end 218.75 98) (width 0.4) (layer "F.Cu") (net 48))
-  (segment (start 213.8625 95) (end 215.75 95) (width 0.4) (layer "F.Cu") (net 48))
-  (segment (start 218.75 98) (end 218.75 100.7) (width 0.4) (layer "F.Cu") (net 48))
+  (segment (start 220.6 98.9) (end 220.6 100.4) (width 0.4) (layer "F.Cu") (net 48))
+  (segment (start 220.4 98.7) (end 220.6 98.9) (width 0.4) (layer "F.Cu") (net 48))
+  (segment (start 215.8 95) (end 219.5 98.7) (width 0.4) (layer "F.Cu") (net 48))
+  (segment (start 219.5 98.7) (end 220.4 98.7) (width 0.4) (layer "F.Cu") (net 48))
+  (segment (start 213.8625 95) (end 215.8 95) (width 0.4) (layer "F.Cu") (net 48))
   (segment (start 202 208.3125) (end 202 206.4125) (width 0.22) (layer "F.Cu") (net 59))
   (segment (start 200.0325 153.8175) (end 193.6825 153.8175) (width 0.4) (layer "F.Cu") (net 70))
@@
         (xy 205.5 106.25)
         (xy 205.5 102.5)
+        (xy 216.3 102.5)
+        (xy 216.3 98.7)
+        (xy 218.5 98.7)
+        (xy 218.5 102.5)
         (xy 219.75 102.5)
       )
@@
     (polygon
       (pts
-        (xy 216.25 101)
-        (xy 214.25 101)
-        (xy 214.25 98.75)
-        (xy 216.25 98.75)
+        (xy 214.9 101)
+        (xy 212.9 101)
+        (xy 212.9 98.75)
+        (xy 214.9 98.75)
       )
     )
