File: NR1B-SQT56/NR1B-SQT56.kicad_sch (KiCad schematic)
At the start: 45 parts, among them J1 Conn_02x04_Odd_Even, J2 Conn_02x04_Odd_Even, U1 DG419LDY, U2 OPA189ID, U3 NCV7800, U4 NCV8114ASN120T1G, U5 S29GL01GP, U6 OPA189ID, U7 Lattice_HX1K-CB132, X1 NUCLEO144-ZIO

Commit message: FPGA schematic functional
Parts:
- removed C11, C12, C13, C15, C17, C18, C2, C20, C21, C3, C4, C5, C6, C7, C9: 0.1uF, Capacitor_SMD:C_0805_2012Metric, symbol Device:C
- removed U7: Lattice_HX1K-CB132, NISoC-Socket:Lattice_CB132-iCE, symbol NISoC-Socket:Lattice_HX1K-CB132
- added D10, D11, D12, D13, D14, D15, D17, D18, D7, D8, D9: ESDA6V1BC6, Package_TO_SOT_SMD:SOT-23-6, symbol NISoC-Socket:ESDA6V1BC6
- added D16: ESDA25-4BP6, Package_TO_SOT_SMD:SOT-23-6, symbol NISoC-Socket:ESDA25-4BP6
- added R3, R4: 1M, Resistor_SMD:R_0805_2012Metric, symbol Device:R
- J1, J2: value Conn_02x04_Odd_Even -> 0.1" Female Long Tail
Connections:
- net +15V: now also D3.1 (K), D5.1 (K); no longer D3.2 (A), D5.2 (A)
- net +15V_IN: now also D3.2 (A); no longer D3.1 (K)
- net +3.3V: now also D16.6; no longer U5.53 (~{BYTE})
- net -15V: now also U1.7 (V-)
- net A0: now also D11.6
- net A1: now also D11.4
- net A10: now also D7.3
- net A11: now also D7.1
- net A12: now also D12.6
- net A13: now also D12.4
- net A14: now also D12.3
- net A15: now also D12.1
- net A16: now also D10.6
- net A17: now also D10.4
- net A18: now also D10.3
- net A19: now also D10.1
- net A2: now also D11.3
- net A20: now also D8.6
- net A21: now also D8.4
- net A22: now also D8.3
- net A23: now also D8.1
- net A3: now also D11.1
- net A4: now also D9.6
- net A5: now also D9.4
- net A6: now also D9.3
- net A7: now also D9.1
- net A8: now also D7.6
- net A9: now also D7.4
- net ANA_VWL: now also R3.1
- net ANA_WP: now also NT1.1, R4.1; no longer NT1.2
- net ANA_WP_SENSE: now also NT1.2; no longer NT1.1
- net DQ0: now also D13.1
- net DQ1: now also D13.3
- net DQ10: now also D17.4
- net DQ11: now also D17.6
- net DQ12: now also D18.1
- net DQ13: now also D18.3
- net DQ14: now also D18.4
- net DQ15: now also D18.6
- net DQ2: now also D13.4
- net DQ3: now also D13.6
- net DQ4: now also D15.1
- net DQ5: now also D15.3
- net DQ6: now also D15.4
- net DQ7: now also D15.6
- net DQ8: now also D17.1
- net DQ9: now also D17.3
- net GND: now also D5.2 (A), D10.2 (C), D10.5 (C), D11.2 (C), D11.5 (C), D12.2 (C), D12.5 (C), D13.2 (C), D14.2 (C), D15.2 (C), D15.5 (C), D16.2 (C), D16.5 (C), D17.2 (C), D17.5 (C), D18.2 (C), D18.5 (C), D7.2 (C), D7.5 (C), D8.2 (C), D8.5 (C), D9.2 (C), D9.5 (C), R3.2, R4.2; no longer D5.1 (K), U1.7 (V-), X1.104 (AGND)
- net RY/~{BY}: now also D14.6
- net WP_BUF: now also D16.3
- net VWL_BUF: now reaches U5.14 (~{RESET}), U6.2 (-), U6.6
- net VWL_BUF: now also D16.4
- net QSPI.IO2: now reaches X1.11 (PF7)
- net QSPI.SCK: now reaches X1.114 (PF10)
- net ~{MCU_RESET}: now reaches X1.14 (~{RST})
- net QSPI.IO1: now reaches X1.54 (PF8)
- net QSPI.IO0: now reaches X1.56 (PF9)
- net QSPI.IO3: now reaches X1.9 (PF6)
- net QSPI.~{CS}: now reaches X1.97 (PB10)
- net ~{FPGA_CE} renamed FC.~{CE}
- net FC.~{CE}: now also D16.1
- net ~{OE} renamed FC.~{OE}
- net FC.~{OE}: now also D14.1
- net ~{WE} renamed FC.~{WE}
- net FC.~{WE}: now also D14.3
- new net: D13.5 (C), D14.5 (C)
- new net FC.~{BYTE}: D14.4, U5.53 (~{BYTE})
- no-connect marks 181 -> 124
Other:
- added sheet FPGA (NR1B-SQT56-FPGA.kicad_sch)
- note added: "1V2"
- note added: "9V"
- note added: "Optional discharge resistor"
- note added: "Power"
- note added: "TODO - Controller QSPI - Power Sequencing - FPGA sheet - Test points"
- note added: "Vwl buffer"
- note added: "WP buffer"
- note removed: "Capacitors"
- note removed: "Detector Interface"
- note removed: "Power Protection"
- note removed: "WP Buffer"
- moved on the sheet: C1, C10, C14, C16, C19, C22, C23, C24, C25, C8, D1, D2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

Commit message: Finish NR1B-SQT56
Parts:
- removed D10, D11, D12, D13, D14, D15, D17, D18, D7, D8, D9: ESDA6V1BC6, Package_TO_SOT_SMD:SOT-23-6, symbol NISoC-Socket:ESDA6V1BC6
- removed D2, D5: 18V, Diode_SMD:D_SOD-323, symbol Device:D
- removed D4: S1G, Diode_SMD:D_SOD-323, symbol Device:D
- removed D6: 5.1V, Diode_SMD:D_SOD-323, symbol Device:D
- added D10, D11, D12, D13, D14, D15, D16, D17, D6, D7, D8, D9: PESD4USB3B_TBS, Package_DFN_QFN:Diodes_UDFN-10_1.0x2.5mm_P0.5mm, symbol NISoC-Socket:PESD4USB3B_TBS
- added D3, D4: 18V, Diode_SMD:D_SOD-323, symbol Device:D_Zener
- added D5: 5.1V, Diode_SMD:D_SOD-323, symbol Device:D_Zener
- added FID1, FID2, FID3: Fiducial, Fiducial:Fiducial_0.5mm_Mask1mm, symbol Mechanical:Fiducial
- added TP1: VWL_BUF, TestPoint:TestPoint_2Pads_Pitch2.54mm_Drill0.8mm, symbol Connector:TestPoint_2Pole
- added TP2: WP_BUF, TestPoint:TestPoint_2Pads_Pitch2.54mm_Drill0.8mm, symbol Connector:TestPoint_2Pole
- added TP3: -15V, TestPoint:TestPoint_2Pads_Pitch2.54mm_Drill0.8mm, symbol Connector:TestPoint_2Pole
- added TP4: +15V, TestPoint:TestPoint_2Pads_Pitch2.54mm_Drill0.8mm, symbol Connector:TestPoint_2Pole
- added TP5: 3.3V, TestPoint:TestPoint_2Pads_Pitch2.54mm_Drill0.8mm, symbol Connector:TestPoint_2Pole
- added TP6: ANA_CE, TestPoint:TestPoint_2Pads_Pitch2.54mm_Drill0.8mm, symbol Connector:TestPoint_2Pole
- added TP7: 1.2V, TestPoint:TestPoint_2Pads_Pitch2.54mm_Drill0.8mm, symbol Connector:TestPoint_2Pole
- added TP8: ~{CE}, TestPoint:TestPoint_2Pads_Pitch2.54mm_Drill0.8mm, symbol Connector:TestPoint_2Pole
- C10: renamed from C23; footprint Capacitor_SMD:C_0805_2012Metric -> Capacitor_SMD:C_0603_1608Metric
- C2: renamed from C25; footprint Capacitor_SMD:C_0805_2012Metric -> Capacitor_SMD:C_0603_1608Metric
- C3: renamed from C14; footprint Capacitor_SMD:C_0805_2012Metric -> Capacitor_SMD:C_0603_1608Metric
- C5: renamed from C16; footprint Capacitor_SMD:C_0805_2012Metric -> Capacitor_SMD:C_0603_1608Metric
- C6: renamed from C19; footprint Capacitor_SMD:C_0805_2012Metric -> Capacitor_SMD:C_0603_1608Metric
- C7: renamed from C24; footprint Capacitor_SMD:C_0805_2012Metric -> Capacitor_SMD:C_0603_1608Metric
- C8: renamed from C1; footprint Capacitor_SMD:C_0805_2012Metric -> Capacitor_SMD:C_0603_1608Metric
- C9: renamed from C22; footprint Capacitor_SMD:C_0805_2012Metric -> Capacitor_SMD:C_0603_1608Metric
- D1: value D -> S1G; footprint Diode_SMD:D_SOD-323 -> Diode_SMD:D_SMA
- D2: renamed from D3; footprint Diode_SMD:D_SOD-323 -> Diode_SMD:D_SMA
- renumbered C10 to C1, C8 to C4, D16 to D18, NT2 to NT1, NT1 to NT2, U6 to U1, U1 to U5, U5 to U6
Connections:
- net 3.3V_IN is gone; now on net +3.3V: X1.16 (+3V3)
- net +15V: now also D4.1 (K), TP4.1
- net +1V2: now also TP7.2
- net +3.3V: now also D5.1 (K), TP5.1
- net -15V: now also D3.2 (A), TP3.1; no longer U5.7 (V-)
- net A0: now also D16.5, D16.6
- net A1: now also D9.5, D9.6
- net A10: now also D8.2, D8.9
- net A11: now also D11.4, D11.7
- net A12: now also D6.4, D6.7
- net A13: now also D8.4, D8.7
- net A14: now also D11.2, D11.9
- net A15: now also D6.5, D6.6
- net A16: now also D12.5, D12.6
- net A17: now also D10.2, D10.9
- net A18: now also D7.4, D7.7
- net A19: now also D8.1, D8.10
- net A2: now also D10.5, D10.6
- net A20: now also D6.1, D6.10
- net A21: now also D7.5, D7.6
- net A22: now also D8.5, D8.6
- net A23: now also D11.1, D11.10
- net A24: now also D16.1, D16.10
- net A25: now also D14.5, D14.6
- net A3: now also D7.1, D7.10
- net A4: now also D9.4, D9.7
- net A5: now also D10.4, D10.7
- net A6: now also D7.2, D7.9
- net A7: now also D9.2, D9.9
- net A8: now also D11.5, D11.6
- net A9: now also D6.2, D6.9
- net ANA_CE: now also TP6.1
- net DQ0: now also D17.2, D17.9
- net DQ1: now also D16.2, D16.9
- net DQ10: now also D14.1, D14.10
- net DQ11: now also D13.5, D13.6
- net DQ12: now also D12.1, D12.10
- net DQ13: now also D15.2, D15.9
- net DQ14: now also D14.4, D14.7
- net DQ15: now also D12.4, D12.7
- net DQ2: now also D13.4, D13.7
- net DQ3: now also D15.5, D15.6
- net DQ4: now also D15.4, D15.7
- net DQ5: now also D14.2, D14.9
- net DQ6: now also D12.2, D12.9
- net DQ7: now also D17.4, D17.7
- net DQ8: now also D13.2, D13.9
- net DQ9: now also D17.1, D17.10
- net FC.~{BYTE}: now also D17.5, D17.6
- net FC.~{CE}: no longer D18.1
- net FC.~{OE}: now also D16.4, D16.7
- net FC.~{WE}: now also D10.1, D10.10
- net GND: now also U5.7 (V-), D10.3 (C), D10.8 (C), D11.3 (C), D11.8 (C), D12.3 (C), D12.8 (C), D13.1, D13.10, D13.3 (C), D13.8 (C), D14.3 (C), D14.8 (C), D15.1, D15.10, D15.3 (C), D15.8 (C), D16.3 (C), D16.8 (C), D17.3 (C), D17.8 (C), D3.1 (K), D4.2 (A), D5.2 (A), D6.3 (C), D6.8 (C), D7.3 (C), D7.8 (C), D8.3 (C), D8.8 (C), D9.3 (C), D9.8 (C), TP1.2, TP2.2, TP3.2, TP4.2, TP5.2, TP6.2, TP7.1, TP8.1
- net RY/~{BY}: now also D9.1, D9.10
- net VWL_BUF: now also TP1.1
- net WP_BUF: now also TP2.1
- net ~{CE}: now also D18.1, TP8.2
Other:
- sheet FPGA ports: added { DQ[0..15] A[0..25] }; removed A[0..25], DQ[0..15]
- note added: "Connectors"
- note added: "ESD Protection"
- note added: "ESD Protection to protect FPGA"
- note removed: "TODO - Controller QSPI - Power Sequencing - FPGA sheet - Test points"
- moved on the sheet: C1, C10, C2, C3, C4, C5, C6, C7, C8, C9, D1, D18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
