File: NR1B-SQT56/NR1B-SQT56.kicad_pcb (KiCad board)
At the start: 4 copper layers, 70.5 x 134 mm, 45 parts, among them J1 Conn_02x04_Odd_Even, J2 Conn_02x04_Odd_Even, U1 DG419LDY, U2 OPA189ID, U3 NCV7800, U4 NCV8114ASN120T1G, U5 S29GL01GP, U6 OPA189ID, U7 Lattice_HX1K-CB132, X1 NUCLEO144-ZIO

Commit message: Finish NR1B-SQT56
Parts:
- added C26: 0.1uF, Capacitor_SMD:C_0402_1005Metric, B.Cu at (93.7, 124.3)
- added C27: 0.1uF, Capacitor_SMD:C_0402_1005Metric, F.Cu at (96.2, 118.9)
- added C28: 0.1uF, Capacitor_SMD:C_0402_1005Metric, B.Cu at (90.5, 124.6)
- added C29: 0.1uF, Capacitor_SMD:C_0402_1005Metric, B.Cu at (98.8, 125.9)
- added C30: 0.1uF, Capacitor_SMD:C_0402_1005Metric, B.Cu at (94.1, 129.5)
- added D10: PESD4USB3B_TBS, Package_DFN_QFN:Diodes_UDFN-10_1.0x2.5mm_P0.5mm, F.Cu at (86.2, 112.4)
- added D11: PESD4USB3B_TBS, Package_DFN_QFN:Diodes_UDFN-10_1.0x2.5mm_P0.5mm, F.Cu at (89.4, 112.4)
- added D12: PESD4USB3B_TBS, Package_DFN_QFN:Diodes_UDFN-10_1.0x2.5mm_P0.5mm, F.Cu at (100.2, 112.5)
- added D13: PESD4USB3B_TBS, Package_DFN_QFN:Diodes_UDFN-10_1.0x2.5mm_P0.5mm, F.Cu at (103.4, 112.5)
- added D14: PESD4USB3B_TBS, Package_DFN_QFN:Diodes_UDFN-10_1.0x2.5mm_P0.5mm, F.Cu at (106.6, 112.5)
- added D15: PESD4USB3B_TBS, Package_DFN_QFN:Diodes_UDFN-10_1.0x2.5mm_P0.5mm, F.Cu at (116.2, 112.5)
- added D16: PESD4USB3B_TBS, Package_DFN_QFN:Diodes_UDFN-10_1.0x2.5mm_P0.5mm, F.Cu at (109.8, 112.5)
- added D17: PESD4USB3B_TBS, Package_DFN_QFN:Diodes_UDFN-10_1.0x2.5mm_P0.5mm, F.Cu at (113.0, 112.5)
- added D18: ESDA25-4BP6, Package_TO_SOT_SMD:SOT-23-6, B.Cu at (88.7, 89.5)
- added D19: GREEN, LED_SMD:LED_0805_2012Metric, F.Cu at (116.6, 172.1)
- added D20: D, Diode_SMD:D_SOD-323, F.Cu at (76.0, 163.8)
- added D21: PESD4USB3B_TBS, Package_DFN_QFN:Diodes_UDFN-10_1.0x2.5mm_P0.5mm, F.Cu at (85.0, 138.2)
- added D22: PESD4USB3B_TBS, Package_DFN_QFN:Diodes_UDFN-10_1.0x2.5mm_P0.5mm, F.Cu at (85.0, 143.3)
- added D23: PESD4USB3B_TBS, Package_DFN_QFN:Diodes_UDFN-10_1.0x2.5mm_P0.5mm, F.Cu at (85.0, 153.5)
- added D24: PESD4USB3B_TBS, Package_DFN_QFN:Diodes_UDFN-10_1.0x2.5mm_P0.5mm, F.Cu at (85.0, 158.7)
- added D27: PESD4USB3B_TBS, Package_DFN_QFN:Diodes_UDFN-10_1.0x2.5mm_P0.5mm, F.Cu at (106.5, 144.6)
- added D28: PESD4USB3B_TBS, Package_DFN_QFN:Diodes_UDFN-10_1.0x2.5mm_P0.5mm, F.Cu at (106.5, 154.8)
- added D7: PESD4USB3B_TBS, Package_DFN_QFN:Diodes_UDFN-10_1.0x2.5mm_P0.5mm, F.Cu at (76.6, 112.4)
- added D8: PESD4USB3B_TBS, Package_DFN_QFN:Diodes_UDFN-10_1.0x2.5mm_P0.5mm, F.Cu at (79.8, 112.4)
- added D9: PESD4USB3B_TBS, Package_DFN_QFN:Diodes_UDFN-10_1.0x2.5mm_P0.5mm, F.Cu at (83.0, 112.4)
- added FID1: Fiducial, Fiducial:Fiducial_0.5mm_Mask1mm, F.Cu at (62.3, 45.3)
- added FID2: Fiducial, Fiducial:Fiducial_0.5mm_Mask1mm, F.Cu at (129.2, 45.3)
- added FID3: Fiducial, Fiducial:Fiducial_0.5mm_Mask1mm, F.Cu at (129.2, 175.5)
- added J3: Conn_01x07, Connector_PinHeader_2.54mm:PinHeader_1x07_P2.54mm_Vertical, F.Cu at (119.3, 120.9)
- added J4: Conn_02x10_Odd_Even, Connector_PinHeader_2.54mm:PinHeader_2x10_P2.54mm_Vertical, F.Cu at (79.0, 137.0)
- added J5: Conn_02x10_Odd_Even, Connector_PinHeader_2.54mm:PinHeader_2x10_P2.54mm_Vertical, F.Cu at (110.0, 137.0)
- added JP1: 0.1" Header, Connector_PinHeader_2.54mm:PinHeader_1x02_P2.54mm_Vertical, F.Cu at (83.2, 170.0)
- added R10: 10k, Resistor_SMD:R_0603_1608Metric, F.Cu at (98.9, 133.4)
- added R11: 10k, Resistor_SMD:R_0603_1608Metric, F.Cu at (79.5, 163.8)
- added R3: 1M, Resistor_SMD:R_0805_2012Metric, F.Cu at (120.0, 65.0)
- added R4: 1M, Resistor_SMD:R_0805_2012Metric, F.Cu at (120.0, 60.0)
- added R5: 100, Resistor_SMD:R_0603_1608Metric, B.Cu at (100.5, 127.8)
- added R6: 100, Resistor_SMD:R_0603_1608Metric, B.Cu at (88.5, 118.8)
- added R7: 10k, Resistor_SMD:R_0603_1608Metric, F.Cu at (116.6, 168.3)
- added R8: 5, Resistor_SMD:R_0603_1608Metric, F.Cu at (100.0, 134.5)
- added R9: 10k, Resistor_SMD:R_0603_1608Metric, F.Cu at (118.6, 168.3)
- added SW1: Push Button, NISoC-Socket:TE_1-1571636-0, F.Cu at (74.5, 171.0)
- added TP1: VWL_BUF, TestPoint:TestPoint_2Pads_Pitch2.54mm_Drill0.8mm, F.Cu at (95.2, 83.0)
- added TP10: IOR_109, TestPoint:TestPoint_THTPad_D1.5mm_Drill0.7mm, F.Cu at (120.6, 117.0)
- added TP11: IOT_188, TestPoint:TestPoint_THTPad_D1.5mm_Drill0.7mm, F.Cu at (86.5, 117.3)
- added TP2: WP_BUF, TestPoint:TestPoint_2Pads_Pitch2.54mm_Drill0.8mm, F.Cu at (98.8, 83.0)
- added TP3: -15V, TestPoint:TestPoint_2Pads_Pitch2.54mm_Drill0.8mm, F.Cu at (91.1, 46.9)
- added TP4: +15V, TestPoint:TestPoint_2Pads_Pitch2.54mm_Drill0.8mm, F.Cu at (91.1, 49.4)
- added TP5: 3.3V, TestPoint:TestPoint_2Pads_Pitch2.54mm_Drill0.8mm, F.Cu at (97.1, 144.5)
- added TP6: ANA_CE, TestPoint:TestPoint_2Pads_Pitch2.54mm_Drill0.8mm, F.Cu at (108.4, 70.6)
- added TP7: 1.2V, TestPoint:TestPoint_2Pads_Pitch2.54mm_Drill0.8mm, F.Cu at (94.6, 147.0)
- added TP8: ~{CE}, TestPoint:TestPoint_2Pads_Pitch2.54mm_Drill0.8mm, F.Cu at (119.9, 109.6)
- added TP9: CDONE, TestPoint:TestPoint_2Pads_Pitch2.54mm_Drill0.8mm, F.Cu at (117.8, 163.6)
- added U8: W25Q128JVS, Package_SO:SOIC-8_5.23x5.23mm_P1.27mm, F.Cu at (107.6, 123.9)
- added Y1: SiT2001, Package_TO_SOT_SMD:SOT-23-5, F.Cu at (98.0, 130.7)
- C1: value 0.1uF -> 0.33uF; moved to F.Cu
- C10: value 0.33uF -> 0.1uF; footprint Capacitor_SMD:C_0805_2012Metric -> Capacitor_SMD:C_0603_1608Metric
- C11, C12: value 0.1uF -> 10uF
- C13, C14, C2, C3, C9: footprint Capacitor_SMD:C_0805_2012Metric -> Capacitor_SMD:C_0603_1608Metric
- C15, C6, C7: value 0.1uF -> 1uF; footprint Capacitor_SMD:C_0805_2012Metric -> Capacitor_SMD:C_0603_1608Metric; moved to F.Cu
- C16, C17, C5: footprint Capacitor_SMD:C_0805_2012Metric -> Capacitor_SMD:C_0603_1608Metric; moved to F.Cu
- C18, C23, C25: footprint Capacitor_SMD:C_0805_2012Metric -> Capacitor_SMD:C_0402_1005Metric; moved to F.Cu
- C19: value 1uF -> 0.1uF; footprint Capacitor_SMD:C_0805_2012Metric -> Capacitor_SMD:C_0402_1005Metric; moved to F.Cu
- C20, C21, C22: footprint Capacitor_SMD:C_0805_2012Metric -> Capacitor_SMD:C_0402_1005Metric
- C24: value 1uF -> 0.1uF; footprint Capacitor_SMD:C_0805_2012Metric -> Capacitor_SMD:C_0402_1005Metric
- C4: value 0.1uF -> 47uF 16V; footprint Capacitor_SMD:C_0805_2012Metric -> Capacitor_SMD:CP_Elec_5x5.3; moved to F.Cu
- C8: value 47uF 16V -> 0.1uF; footprint Capacitor_SMD:CP_Elec_5x5.3 -> Capacitor_SMD:C_0603_1608Metric; moved to B.Cu
- D1: value D -> S1G; footprint Diode_SMD:D_SOD-323 -> Diode_SMD:D_SMA; moved to F.Cu
- D2: value 18V -> S1G; footprint Diode_SMD:D_SOD-323 -> Diode_SMD:D_SMA; moved to F.Cu
- D3, D4: value S1G -> 18V; moved to F.Cu
- D5: value 18V -> 5.1V; moved to F.Cu
- D6: value 5.1V -> PESD4USB3B_TBS; footprint Diode_SMD:D_SOD-323 -> Package_DFN_QFN:Diodes_UDFN-10_1.0x2.5mm_P0.5mm; moved to F.Cu
- J1, J2: value Conn_02x04_Odd_Even -> 0.1" Female Long Tail
- U1: value DG419LDY -> OPA189ID; footprint Package_SO:SOIC-8_3.9x4.9mm_P1.27mm -> Package_SO:VSSOP-8_3.0x3.0mm_P0.65mm
- U3, U4: moved to F.Cu
- U5: value S29GL01GP -> DG419LDY; footprint NISoC-Socket:Socket_TSOP-56 -> Package_SO:SOIC-8_3.9x4.9mm_P1.27mm; moved to B.Cu
- U6: value OPA189ID -> S29GL01GP; footprint Package_SO:VSSOP-8_3.0x3.0mm_P0.65mm -> NISoC-Socket:Socket_TSOP-56; moved to F.Cu
- U7: value Lattice_HX1K-CB132 -> Lattice_HX8K-CB132; moved to F.Cu
- moved NT1 135.8 mm to (83.4, 85.4)
- moved U1 128.0 mm to (80.5, 84.8), turned to -90 degrees
- moved U6 126.8 mm to (77.1, 92.5), turned to 0 degrees
- moved R1 126.8 mm to (87.8, 100.1), turned to -90 degrees
- moved C17 126.0 mm to (76.2, 166.2)
- moved NT2 123.8 mm to (95.3, 101.9), turned to 0 degrees
- moved C14 121.2 mm to (91.1, 121.5), turned to -135 degrees
- moved U2 120.2 mm to (92.5, 98.5)
- moved R2 118.5 mm to (92.0, 102.0), turned to -90 degrees
- moved C4 113.6 mm to (72.1, 127.0), turned to 90 degrees
- moved C16 113.3 mm to (103.8, 122.4), turned to 90 degrees
- moved D4 111.5 mm to (81.1, 56.2), turned to 0 degrees
- moved D6 108.0 mm to (73.4, 112.4), turned to -90 degrees
- moved C2 106.7 mm to (77.5, 84.8), turned to 90 degrees
- moved D1 106.7 mm to (73.6, 49.0), turned to 0 degrees
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Connections:
- net -15V_IN renamed /-15V_IN
- C1 pad 1: GND -> +15V
- C1 pad 2: +3.3V -> GND
- C10 pad 1: +15V -> +3.3V
- C11 pad 1: +3.3V -> /FPGA/VCCPLL0
- C11 pad 2: GND -> /FPGA/GNDPLL0
- C12 pad 1: +3.3V -> /FPGA/VCCPLL1
- C12 pad 2: GND -> /FPGA/GNDPLL1
- C13 pad 1: +1V2 -> /FPGA/VCCPLL0
- C13 pad 2: GND -> /FPGA/GNDPLL0
- C14 pad 1: +15V -> /FPGA/VCCPLL1
- C14 pad 2: -15V -> /FPGA/GNDPLL1
- C15 pad 1: +3.3V -> GND
- C15 pad 2: GND -> /FPGA/CLK_VDD
- C16 pad 1: ANA_CE -> GND
- C16 pad 2: GND -> +3.3V
- C17 pad 1: +1V2 -> /FPGA/~{CRESET}
- C2 pad 1: +3.3V -> +15V
- C2 pad 2: GND -> -15V
- C20 pad 1: +3.3V -> +1V2
- C21 pad 1: +1V2 -> +3.3V
- C22 pad 1: +3.3V -> +1V2
- C25 pad 1: +15V -> +3.3V
- C25 pad 2: -15V -> GND
- C3 pad 1: +3.3V -> +15V
- C3 pad 2: GND -> -15V
- C4 pad 1: +1V2 -> +3.3V
- C5 pad 1: +3.3V -> /ANA_CE
- C6 pad 1: +1V2 -> +3.3V
- C7 pad 1: +3.3V -> +1V2
- C8 pad 1: +3.3V -> GND
- C8 pad 2: GND -> +3.3V
- C9 pad 1: +1V2 -> +3.3V
- D2 pad 1: GND -> +15V
- D2 pad 2: -15V -> /+15V_IN
- D3 pad 1: +15V_IN -> GND
- D3 pad 2: +15V -> -15V
- D4 pad 1: +3.3V -> +15V
- D4 pad 2: 3.3V_IN -> GND
- D5 pad 1: GND -> +3.3V
- D5 pad 2: +15V -> GND
- D6 pad 1: +3.3V -> /FPGA/A20
- D6 pad 2: GND -> /FPGA/A9
- J1 pad 1: ANA_WP_SENSE -> /ANA_WP_SENSE
- J1 pad 3: ANA_WP -> /ANA_WP
- J1 pad 5: ANA_VWL_SENSE -> /ANA_VWL_SENSE
- J1 pad 7: ANA_VWL -> /ANA_VWL
- J2 pad 2: +15V_IN -> /+15V_IN
- NT1 pad 1: ANA_WP_SENSE -> /ANA_VWL_SENSE
- NT1 pad 2: ANA_WP -> /ANA_VWL
- NT2 pad 1: ANA_VWL_SENSE -> /ANA_WP
- NT2 pad 2: ANA_VWL -> /ANA_WP_SENSE
- R1 pad 1: WP_BUF -> /WP_BUF
- U1 pad 1: /~{CE} -> unconnected-(U1-Pad1)
- U1 pad 2: ANA_CE -> /VWL_BUF
- U1 pad 3: GND -> /ANA_VWL
- U1 pad 4: +15V -> -15V
- U1 pad 5: +3.3V -> unconnected-(U1-Pad5)
- U1 pad 6: /CE_SW -> /VWL_BUF
- U1 pad 7: GND -> +15V
- U1 pad 8: /~{FPGA_CE} -> unconnected-(U1-Pad8)
- U2 pad 1: (no net) -> unconnected-(U2-Pad1)
- U2 pad 3: ANA_WP -> /ANA_WP
- U2 pad 5: (no net) -> unconnected-(U2-Pad5)
- U2 pad 6: WP_BUF -> /WP_BUF
- U2 pad 8: (no net) -> unconnected-(U2-Pad8)
- U3 pad 3: ANA_CE -> /ANA_CE
- U5 pad 1: /A23 -> /~{CE}
- U5 pad 2: /A22 -> /ANA_CE
- U5 pad 3: /A15 -> GND
- U5 pad 4: /A14 -> +15V
- U5 pad 5: /A13 -> +3.3V
- U5 pad 6: /A12 -> /CE_SW
- U5 pad 7: /A11 -> GND
- U5 pad 8: /A10 -> /FC.~{CE}
- U6 pad 1: (no net) -> /FPGA/A23
- U6 pad 2: Net-(U5-Pad14) -> /FPGA/A22
- U6 pad 3: ANA_VWL -> /FPGA/A15
- U6 pad 4: -15V -> /FPGA/A14
- U6 pad 5: (no net) -> /FPGA/A13
- U6 pad 6: Net-(U5-Pad14) -> /FPGA/A12
- U6 pad 7: +15V -> /FPGA/A11
- U6 pad 8: (no net) -> /FPGA/A10
- U7 pad A1: /DQ15 -> /FPGA/A6
- U7 pad A10: /A22 -> /FPGA/A2
- U7 pad A11: (no net) -> /FPGA/A5
- U7 pad A12: /A8 -> /FPGA/A23
- U7 pad A13: /A23 -> unconnected-(U7-PadA13)
- U7 pad A14: /A14 -> +3.3V
- U7 pad A2: unconnected-(U7-PadA2) -> /FPGA/A3
- U7 pad A3: (no net) -> /FPGA/A22
- U7 pad A4: /DQ13 -> /FPGA/A13
- U7 pad A5: /DQ7 -> /FPGA/A10
- U7 pad A6: /A24 -> /FPGA/A19
- U7 pad A7: unconnected-(U7-PadA7) -> /FPGA/A1
- U7 pad A8: (no net) -> +3.3V
- U7 pad B1: unconnected-(U7-PadB1) -> /FPGA/A12
- U7 pad B14: /A11 -> /FPGA/A16
- U7 pad C1: /A16 -> /FPGA/A15
- U7 pad C10: unconnected-(U7-PadC10) -> /FPGA/A17
- U7 pad C11: /A21 -> /FPGA/A8
- U7 pad C12: /A15 -> /FPGA/A11
- U7 pad C14: /A17 -> /FPGA/DQ11
- U7 pad C3: /A25 -> unconnected-(U7-PadC3)
- U7 pad C4: unconnected-(U7-PadC4) -> /FPGA/A21
- U7 pad C5: unconnected-(U7-PadC5) -> /FPGA/A20
- U7 pad C6: unconnected-(U7-PadC6) -> /FPGA/A4
- U7 pad C7: unconnected-(U7-PadC7) -> /RY/~{BY}
- U7 pad C8: unconnected-(U7-PadC8) -> /FPGA/VCCPLL1
- U7 pad D1: unconnected-(U7-PadD1) -> /FPGA/IOL_5+
- U7 pad D10: unconnected-(U7-PadD10) -> /FC.~{WE}
- U7 pad D11: unconnected-(U7-PadD11) -> /FPGA/A14
- U7 pad D12: /A12 -> /FPGA/DQ15
- U7 pad D14: /~{WE} -> /FPGA/DQ2
- U7 pad D3: /DQ4 -> unconnected-(U7-PadD3)
- U7 pad D5: unconnected-(U7-PadD5) -> /FPGA/A9
- U7 pad D6: unconnected-(U7-PadD6) -> /FPGA/A18
- U7 pad D7: unconnected-(U7-PadD7) -> /FPGA/A7
- U7 pad D8: unconnected-(U7-PadD8) -> /FPGA/GNDPLL1
- U7 pad D9: unconnected-(U7-PadD9) -> /FPGA/IOT_188
- U7 pad E1: /DQ6 -> /FPGA/IOL_5-
- U7 pad E11: unconnected-(U7-PadE11) -> /FPGA/DQ6
- U7 pad E12: unconnected-(U7-PadE12) -> /FPGA/DQ12
- U7 pad E14: /A5 -> /FPGA/DQ8
- U7 pad F11: unconnected-(U7-PadF11) -> /FPGA/A25
- U7 pad F12: unconnected-(U7-PadF12) -> /FPGA/DQ14
- U7 pad F14: /A13 -> /FPGA/DQ5
- U7 pad F3: /DQ8 -> /FPGA/IOL_9-
- U7 pad F4: unconnected-(U7-PadF4) -> /FPGA/IOL_9+
- U7 pad G1: /DQ12 -> /FPGA/IOL_13-
- U7 pad G11: unconnected-(U7-PadG11) -> /FPGA/A0
- U7 pad G12: /A18 -> /FC.~{OE}
- U7 pad G14: /A10 -> /FPGA/DQ10
- U7 pad G3: unconnected-(U7-PadG3) -> /FPGA/IOL_13+
- U7 pad H1: /DQ11 -> /FPGA/IOL_14+
- U7 pad H11: unconnected-(U7-PadH11) -> /FPGA/A24
- U7 pad H12: /A19 -> /FPGA/DQ1
- U7 pad H3: unconnected-(U7-PadH3) -> /FPGA/IOL_14-
- U7 pad J1: /DQ3 -> /FPGA/IOL_12-
- U7 pad J12: /RY/~{BY} -> /FPGA/DQ7
- U7 pad J3: /DQ10 -> /FPGA/IOL_12+
- U7 pad K11: unconnected-(U7-PadK11) -> /FC.~{CE}
- U7 pad K12: /BYTE -> /FPGA/DQ0
- U7 pad K14: /A2 -> /FC.~{BYTE}
- U7 pad K3: /DQ5 -> /FPGA/IOL_18+
- U7 pad K4: unconnected-(U7-PadK4) -> /FPGA/IOL_18-
- U7 pad L1: /DQ2 -> /FPGA/IOL_23+
- U7 pad L10: unconnected-(U7-PadL10) -> /FPGA/~{CRESET}
- U7 pad L12: /A4 -> /FPGA/DQ9
- U7 pad L14: /VSS -> /FPGA/DQ3
- U7 pad L4: unconnected-(U7-PadL4) -> /QSPI.~{CS}
- U7 pad L5: /VIO -> /QSPI.SCK
- U7 pad L7: unconnected-(U7-PadL7) -> /FPGA/GNDPLL0
- U7 pad L8: unconnected-(U7-PadL8) -> /FPGA/IOB_87
- U7 pad L9: unconnected-(U7-PadL9) -> /FPGA/IOB_103_CBSEL0
- U7 pad M1: unconnected-(U7-PadM1) -> /FPGA/IOL_23-
- U7 pad M10: unconnected-(U7-PadM10) -> /FPGA/CDONE
- U7 pad M11: unconnected-(U7-PadM11) -> /FPGA/FLASH.DO_IO1
- U7 pad M12: /A9 -> /FPGA/IOR_109
- U7 pad M14: (no net) -> unconnected-(U7-PadM14)
- U7 pad M3: unconnected-(U7-PadM3) -> /QSPI.IO0
- U7 pad M4: /DQ9 -> /QSPI.IO1
- U7 pad M7: /~{OE} -> unconnected-(U7-PadM7)
- U7 pad M8: /A3 -> /FPGA/VCCPLL0
- U7 pad M9: /A6 -> /FPGA/IOB_91
- U7 pad N1: +1V2 -> /FPGA/IOL_25+
- U7 pad N14: /A7 -> /FPGA/DQ4
- U7 pad P1: GND -> /FPGA/IOL_25-
- U7 pad P10: unconnected-(U7-PadP10) -> /FPGA/IOB_104_CBSEL1
- U7 pad P11: unconnected-(U7-PadP11) -> /FPGA/FLASH.DI_IO0
- U7 pad P12: unconnected-(U7-PadP12) -> /FPGA/FLASH.~{CS}
- U7 pad P13: unconnected-(U7-PadP13) -> /FPGA/FLASH.SCK
- U7 pad P14: /A1 -> /FPGA/DQ13
- U7 pad P2: unconnected-(U7-PadP2) -> /QSPI.IO3
- U7 pad P3: /DQ1 -> /QSPI.IO2
- U7 pad P4: /A0 -> /FPGA/IOB_73
- U7 pad P5: /~{FPGA_CE} -> /FPGA/IOB_74
- U7 pad P7: /DQ0 -> /FPGA/FPGA_CLK
- U7 pad P8: unconnected-(U7-PadP8) -> /FPGA/IOB_82_GBIN4
- U7 pad P9: /A20 -> /FPGA/IOB_89
- X1 pad 104: GND -> unconnected-(X1-Pad104)
- X1 pad 11: unconnected-(X1-Pad11) -> /QSPI.IO2
- X1 pad 114: unconnected-(X1-Pad114) -> /QSPI.SCK
- X1 pad 14: unconnected-(X1-Pad14) -> /~{MCU_RESET}
- X1 pad 145: (no net) -> unconnected-(X1-Pad145)
- X1 pad 146: (no net) -> unconnected-(X1-Pad146)
- X1 pad 147: (no net) -> unconnected-(X1-Pad147)
- X1 pad 148: (no net) -> unconnected-(X1-Pad148)
- X1 pad 16: 3.3V_IN -> +3.3V
- X1 pad 54: unconnected-(X1-Pad54) -> /QSPI.IO1
- X1 pad 56: unconnected-(X1-Pad56) -> /QSPI.IO0
- X1 pad 9: unconnected-(X1-Pad9) -> /QSPI.IO3
- X1 pad 97: unconnected-(X1-Pad97) -> /QSPI.~{CS}
Routing:
- net GND: track 300.6 -> 141.3 mm, vias 13 -> 186
- net +15V: track 0.00 -> 123.4 mm, vias 0 -> 11
- net +3.3V: track 53.1 -> 140.5 mm, vias 9 -> 47
- net /QSPI.IO3: track 0.00 -> 83.0 mm, vias 0 -> 1
- net /CE_SW: track 0.00 -> 82.9 mm, vias 0 -> 2
- net /QSPI.IO2: track 0.00 -> 82.0 mm, vias 0 -> 1
- net /FPGA/~{CRESET}: track 0.00 -> 81.9 mm, vias 0 -> 1
- net /~{MCU_RESET}: track 0.00 -> 77.1 mm, vias 0 -> 1
- net -15V: track 0.00 -> 68.1 mm, vias 0 -> 8
- net /ANA_WP: track 0.00 -> 65.2 mm, vias 0 -> 1
- net /ANA_WP_SENSE: track 0.00 -> 62.7 mm, vias 0 -> 1
- net /QSPI.~{CS}: track 0.00 -> 61.2 mm, vias 0 -> 2
- net /ANA_VWL: track 0.00 -> 61.0 mm
- net /FPGA/CDONE: track 0.00 -> 58.0 mm, vias 0 -> 2
- net /ANA_VWL_SENSE: track 0.00 -> 50.5 mm
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- added copper zone on B.Cu, net +15V
- added copper zone on F.Cu, net +15V
- added copper zone on F.Cu, net +1V2
- added copper zone on In2.Cu, net +1V2
- added copper zone on B.Cu, net +3.3V
- added copper zone on In2.Cu, net +3.3V
- added copper zone on B.Cu, net -15V
- added copper zone on F.Cu, net -15V
- added copper zone on B.Cu, net /FPGA/VCCPLL0
- added copper zone on F.Cu, net GND
- added copper zone on In1.Cu, net GND
- removed copper zone on In1.Cu, net +1V2
- removed copper zone on B.Cu, net GND
Other:
- board size 70.5 x 134 mm -> 70.5 x 133.9 mm
- board text added: "+15V"
- board text added: "-15V"
- board text added: "0.062 in"
- board text added: "0.0762 mm"
- board text added: "0.0762 mm / 0.0762 mm"
- board text added: "1.0uF"
- board text added: "4"
- board text added: "70.5000 mm x 133.9000 mm"
- board text added: "ANA_VWL"
- board text added: "ANA_VWL_SENSE"
- board text added: "ANA_WP"
- board text added: "ANA_WP_SENSE"
- board text added: "BOARD CHARACTERISTICS"
- board text added: "Board Thickness:"
- board text added: "Board overall dimensions:"
- board text added: "C20 C22 C24 C26"
- board text added: "CDONE"
- board text added: "CE_SW"
- board text added: "CFLASH"
- board text added: "Castellated pads:"
- board text added: "Copper Finish:"
- board text added: "Copper Layer Count:"
- board text added: "DI/IO0"
- board text added: "DO/IO1"
- board text added: "ENIG"
- board text added: "Edge card connectors:"
- board text added: "G"
- board text added: "GND"
- board text added: "Impedance Control:"
- board text added: "Min hole diameter:"
- board text added: "Min track/spacing:"
- board text added: "NISoC socket carrier 1 x TSOP-56 QSPI interface"
- board text added: "NR1B-SQT56 Angela Jimenez, Aidan Medcalf 2022 University of Dallas"
- board text added: "No"
- board text added: "Nom. 75Ohm impedance Nom. 150Ohm Diff. imp."
- board text added: "Plated Board Edge:"
- board text added: "QIO0"
- board text added: "QIO1"
- board text added: "QIO2"
- board text added: "QIO3"
- board text added: "QSCK"
- board text added: "RESET"
- board text added: "SCK"
- board text added: "VCC"
- board text added: "~{CS}"
- board text added: "~{MCU_RESET}"
- board text added: "~{QCS}"
- board text added: "~{RST}/IO3"
- board text added: "~{WP}/IO2"

Commit message: Exported fab outputs
Parts:
- U3: value NCV7800 -> NCV7809

Commit message: Updated R8 to be 5.1 ohm
Parts:
- R8: value 5 -> 5.1
- U3: value NCV7809 -> NCV7800
Changed lines of the file:
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@@
       (effects (font (size 1 1) (thickness 0.15)))
     )
-    (fp_text value "5" (at 0 1.43 45) (layer "F.Fab")
+    (fp_text value "5.1" (at 0 1.43 45) (layer "F.Fab")
       (effects (font (size 1 1) (thickness 0.15)))
     )
@@
       (effects (font (size 1 1) (thickness 0.15)))
     )
-    (fp_text value "NCV7809" (at 0 6.65 90) (layer "F.Fab")
+    (fp_text value "NCV7800" (at 0 6.65 90) (layer "F.Fab")
       (effects (font (size 1 1) (thickness 0.15)))
     )
